File: SlimeVRDiyModular.brd (EAGLE design)
At the start: 39.4 x 39.5 mm, 46 parts, among them IC1 FT231XS-R, IC6 DW01A, IC7 LM1117MPX-33NOPB, Q1 MMBT3904-TP, Q2 MMBT3904-TP, Q4 FS8205A, U3 TP4056, U4 ESP32-WROOM-32D, U6 SI2301BDS-T1-E3

Commit message: FEAT: update finish rev1 on board
Parts:
- removed BATT: (no value), pinhead:1X02
- removed IC7: LM1117MPX-33NOPB, LM1117MPX-33NOPB:SOT230P700X180-4N
- removed R18, R19: 47k, AccesControlNFC:ERJH3
- added C1: 100nf, AccesControlNFC:CAPC1608X87N
- added IC2: M3406-ADJ, M3406:SOT95P280X100-5N
- added L1: MLF2012A2R2KT000, MLF2012A2R2KT000:INDC2012X105N
- added R1, R3: 10k, AccesControlNFC:RESC1608X55N
- added R2, R4: 40k2, ERJ-S03F4022V:RESC1608X55N
- added S1: 1825966-1, Switches:SWDIP2_256X170P100
- moved C17 116.1 mm to (28.8, 71.6), turned to 270 degrees
- moved R9 107.3 mm to (40.9, 45.1), turned to 0 degrees
- moved R12 106.6 mm to (38.5, 42.7), turned to 90 degrees
- moved R10 105.5 mm to (34.9, 42.7), turned to 90 degrees
- moved R15 103.3 mm to (22.9, 54.0), turned to 90 degrees
- moved D1 101.6 mm to (25.7, 70.5), turned to 0 degrees
- moved C14 100.3 mm to (35.3, 71.3)
- moved C18 100.0 mm to (18.8, 42.7), turned to 270 degrees
- moved C22 99.3 mm to (28.8, 69.0)
- moved C19 98.5 mm to (19.9, 42.7), turned to 90 degrees
- moved C23 97.6 mm to (28.8, 74.2)
- moved C20 96.0 mm to (21.6, 78.6), turned to 0 degrees
- moved C21 94.4 mm to (21.6, 77.5), turned to 0 degrees
- moved C25 91.6 mm to (21.5, 72.8), turned to 90 degrees
- moved R16 90.4 mm to (20.3, 72.9), turned to 90 degrees
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Connections:
- removed net N$14: BATT_SW.3
- removed net VBAT_RAW: BATT.1, BATT_SW.2
- new net N$1: IC2.3, L1.1
- new net N$3: IC2.5, R1.1, R2.1
- net +5V: now also BATT_SW.2, C1.2, IC2.1, IC2.4, R4.2; no longer C23.2, D1.C, IC7.3, U6.2
- net 3.3V: now also JP1.2, L1.2, P2.4, R2.2; no longer IC7.2, IC7.4
- net D34: now also R3.1, R4.1; no longer R18.1, R19.1
- net EN: now also S1.2
- net GND: now also C1.1, IC2.2, JP1.3, JP1.7, P2.1, R1.2, R3.2, S1.1; no longer IC7.1, R19.2
- net SCL: now also JP1.4, P2.2
- net SDA: now also JP1.5, P2.3
- net VBAT+: now also P1.2; no longer BATT_SW.1, R18.2
- net VBAT-: now also P1.1; no longer BATT.2
- net VCC: now also BATT_SW.1, C23.2, D1.C, U6.2
Routing:
- net 3.3V: track 0.00 -> 94.6 mm, vias 0 -> 4
- net VCC: track 0.00 -> 87.5 mm, vias 0 -> 8
- net SDA: track 0.00 -> 63.7 mm, vias 0 -> 2
- net SCL: track 0.00 -> 62.3 mm, vias 0 -> 4
- net EN: track 0.00 -> 62.0 mm, vias 0 -> 4
- net VBUS: track 0.00 -> 60.4 mm, vias 0 -> 4
- net CBUS1: track 0.00 -> 56.3 mm, vias 0 -> 2
- net VBAT-: track 0.00 -> 55.0 mm, vias 0 -> 5
- net VBAT+: track 0.00 -> 50.0 mm, vias 0 -> 5
- net CBUS2: track 0.00 -> 42.7 mm, vias 0 -> 2
- net U0RXD: track 0.00 -> 36.9 mm, vias 0 -> 2
- net U0TXD: track 0.00 -> 36.8 mm, vias 0 -> 2
- net +5V: track 0.00 -> 35.9 mm, vias 0 -> 4
- net DTR: track 0.00 -> 31.2 mm, vias 0 -> 3
- net 0: track 0.00 -> 31.0 mm, vias 0 -> 2
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- added copper zone on layer 1, net GND
- added copper zone on layer 16, net GND
Other:
- outline, holes or cut-outs redrawn
- board text removed: "PS1"
