File: SlimeVRDiyModular.sch (EAGLE design)
At the start: 46 parts, among them IC1 FT231XS-R, IC6 DW01A, IC7 LM1117MPX-33NOPB, Q1 MMBT3904-TP, Q2 MMBT3904-TP, Q4 FS8205A, U3 TP4056, U4 ESP32-WROOM-32D, U6 SI2301BDS-T1-E3

Commit message: FEAT: update finish rev1 on board
Parts:
- removed BATT: (no value), pinhead:PINHD-1X2
- removed IC7: LM1117MPX-33NOPB, LM1117MPX-33NOPB:LM1117MPX-33NOPB
- removed R18, R19: 47k, AccesControlNFC:ERJ-H3EF3300V
- added C1: 100nf, AccesControlNFC:885012206071
- added IC2: M3406-ADJ, M3406:M3406-ADJ
- added L1: MLF2012A2R2KT000, MLF2012A2R2KT000:MLF2012A2R2KT000
- added R1, R3: 10k, AccesControlNFC:ESR03EZPJ103
- added R2, R4: 40k2, ERJ-S03F4022V:ERJ-S03F4022V
- added S1: 1825966-1, Switches:1825966-1
Connections:
- removed net N$14: BATT_SW.3
- removed net VBAT_RAW: BATT.1, BATT_SW.2
- new net N$1: IC2.SW, L1.1
- new net N$3: IC2.FB, R1.1, R2.1
- net +5V: now also BATT_SW.2, C1.2, IC2.RUN, IC2.VIN, R4.2; no longer C23.2, D1.K, IC7.INPUT, U6.S
- net 3.3V: now also JP1.2, L1.2, P2.4, R2.2; no longer IC7.OUTPUT_1, IC7.OUTPUT_2
- net D34: now also R3.1, R4.1; no longer R18.1, R19.1
- net EN: now also S1.2
- net GND: now also C1.1, IC2.GND, JP1.3, JP1.7, P2.1, R1.2, R3.2, S1.1; no longer IC7.GROUND, R19.2
- net SCL: now also JP1.4, P2.2
- net SDA: now also JP1.5, P2.3
- net VBAT+: now also P1.2; no longer BATT_SW.1, R18.2
- net VBAT-: now also P1.1; no longer BATT.2
- net VCC: now also BATT_SW.1, C23.2, D1.K, U6.S
Other:
- note added: "SLIMEVR BY POSITRON ELEKTRONIK"
- note removed: "BNO055 and BMP280"
- note removed: "ESP32 USB CHARGER"
