File: PCB/EAGLE/SlimeVRDiyModular.sch (EAGLE design)
At the start: 46 parts, among them IC1 FT231XS-R, IC6 DW01A, IC7 LM1117MPX-33NOPB, Q1 MMBT3904-TP, Q2 MMBT3904-TP, Q4 FS8205A, U3 TP4056, U4 ESP32-WROOM-32D, U6 SI2301BDS-T1-E3

Commit message: FEAT: update 3D model, gerber and BOM
Parts:
- removed IC7: LM1117MPX-33NOPB, LM1117MPX-33NOPB:LM1117MPX-33NOPB
- removed R18, R19: 47k, AccesControlNFC:ERJ-H3EF3300V
- added C1: 100nf, AccesControlNFC:885012206071
- added IC2: M3406-ADJ, M3406:M3406-ADJ
- added L1: MLF2012A2R2KT000, MLF2012A2R2KT000:MLF2012A2R2KT000
- added R1, R3: 10k, AccesControlNFC:ESR03EZPJ103
- added R2, R4: 40k2, ERJ-S03F4022V:ERJ-S03F4022V
- renumbered JP1 to IMU, LED1 to TX, LED2 to LED, LED5 to RX, LED6 to STBY, LED7 to CHRG, P2 to EXT, S1 to RESET, U4 to ESP32
Connections:
- removed net BUTTON2: ESP32.IO19
- removed net D2: R9.1
- removed net N$4: IMU.5
- new net LED: ESP32.IO19, R9.1
- new net N$1: IC2.SW, L1.1
- net +5V: now also C1.2, IC2.RUN, IC2.VIN, R4.2; no longer IC7.INPUT
- net 3.3V: now also EXT.4, L1.2, R2.2; no longer IC7.OUTPUT_1, IC7.OUTPUT_2
- net D34: now also R3.1, R4.1; no longer R18.1, R19.1
- net GND: now also C1.1, EXT.1, IC2.GND, R1.2, R3.2; no longer IC7.GROUND, R19.2
- net N$3: now also IC2.FB, R1.1, R2.1; no longer IMU.4
- net SCL: now also EXT.2, IMU.4
- net SDA: now also EXT.3, IMU.5
- net VBAT+: no longer R18.2
Other:
- note added: "SLIMEVR BY POSITRON ELEKTRONIK"
- note removed: "BNO055 and BMP280"
- note removed: "ESP32 USB CHARGER"
