File: PCB/EAGLE/SlimeVRDiyModularV2.brd (EAGLE design)
At the start: 39.4 x 39.5 mm, 50 parts, among them IC1 FT231XS-R, IC2 M3406-ADJ, IC6 DW01A, Q1 MMBT3904-TP, Q2 MMBT3904-TP, Q4 FS8205A, U3 TP4056, U6 SI2301BDS-T1-E3

Commit message: FIX: fix problem on pcb
Parts:
- moved R4 0.63 mm to (30.2, 66.7)
- moved R3 0.18 mm to (30.1, 65.5)
- moved LED 0.13 mm to (42.4, 43.1), turned to 270 degrees
Connections:
- removed net N$27: LED.2, R9.2
- new net N$2: LED.1, R9.2
- new net V+: BATT_SW.1, C23.2, D1.C, U6.2
- net 3.3V: now also LED.2; no longer LED.1
- net VCC: no longer BATT_SW.1, C23.2, D1.C, U6.2
Routing:
- net V+: track 0.00 -> 25.4 mm, vias 0 -> 4
- net VCC: track 87.5 -> 63.6 mm, vias 8 -> 6
- net N$20: track 24.7 -> 39.3 mm
- net VBUS: track 60.4 -> 56.3 mm
- net U0RXD: track 36.9 -> 34.5 mm
- net N$2: track 0.00 -> 1.73 mm
- net N$27: track 1.53 -> 0.00 mm
- net CBUS1: track 56.3 -> 55.0 mm
- net +5V: track 35.9 -> 35.1 mm
- net D34: track 13.7 -> 13.1 mm
