File: PCB/EAGLE/SlimeVRDiyModularV2.sch (EAGLE design)
At the start: 50 parts, among them IC1 FT231XS-R, IC2 M3406-ADJ, IC6 DW01A, Q1 MMBT3904-TP, Q2 MMBT3904-TP, Q4 FS8205A, U3 TP4056, U6 SI2301BDS-T1-E3

Commit message: FIX: fix problem on pcb
Connections:
- removed net N$27: LED.A, R9.2
- new net N$2: LED.K, R9.2
- new net V+: BATT_SW.1, C23.2, D1.K, U6.S
- net 3.3V: now also LED.A; no longer LED.K
- net VCC: no longer BATT_SW.1, C23.2, D1.K, U6.S
Other:
- moved on the sheet: LED
Changed lines of the file:
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@@
 <part name="SUPPLY5" library="DecawaveLibrary" library_urn="urn:adsk.eagle:library:5224885" deviceset="3.3V" device=""/>
 <part name="GND5" library="DecawaveLibrary" library_urn="urn:adsk.eagle:library:5224885" deviceset="GND" device=""/>
-<part name="P+1" library="supply1" library_urn="urn:adsk.eagle:library:371" deviceset="VCC" device=""/>
-<part name="P+3" library="supply1" library_urn="urn:adsk.eagle:library:371" deviceset="VCC" device=""/>
+<part name="P+1" library="supply1" library_urn="urn:adsk.eagle:library:371" deviceset="V+" device=""/>
+<part name="P+3" library="supply1" library_urn="urn:adsk.eagle:library:371" deviceset="V+" device=""/>
 </parts>
 <sheets>
@@
 <attribute name="VALUE" x="122.682" y="101.092" size="1.016" layer="96" rot="R180" align="bottom-center"/>
 </instance>
-<instance part="LED" gate="G$1" x="120.142" y="102.87" smashed="yes" rot="R90">
-<attribute name="NAME" x="122.428" y="103.632" size="1.016" layer="95" rot="R90"/>
-<attribute name="VALUE" x="122.428" y="114.808" size="1.016" layer="96" rot="R90"/>
+<instance part="LED" gate="G$1" x="120.142" y="120.396" smashed="yes" rot="R270">
+<attribute name="NAME" x="121.412" y="119.888" size="1.016" layer="95" rot="R270"/>
+<attribute name="VALUE" x="121.158" y="108.458" size="1.016" layer="96" rot="R270"/>
 </instance>
 <instance part="Q1" gate="G$1" x="51.054" y="41.91" smashed="yes">
@@
 <attribute name="VALUE" x="233.426" y="69.088" size="1.016" layer="96" align="top-center"/>
 </instance>
-<instance part="P+1" gate="VCC" x="144.018" y="62.992" smashed="yes">
-<attribute name="VALUE" x="145.288" y="64.516" size="1.016" layer="96" rot="R180"/>
-</instance>
-<instance part="P+3" gate="VCC" x="150.622" y="98.806" smashed="yes" rot="R90">
-<attribute name="VALUE" x="149.098" y="100.076" size="1.016" layer="96" rot="R270"/>
+<instance part="P+1" gate="1" x="144.018" y="62.992" smashed="yes">
+<attribute name="VALUE" x="145.542" y="65.278" size="1.778" layer="96" rot="R180"/>
+</instance>
+<instance part="P+3" gate="1" x="150.622" y="98.806" smashed="yes" rot="R90">
+<attribute name="VALUE" x="148.336" y="100.33" size="1.778" layer="96" rot="R270"/>
 </instance>
 </instances>
@@
 <pinref part="P+8" gate="VCC" pin="VCC"/>
 </segment>
-<segment>
-<pinref part="D1" gate="G$1" pin="K"/>
-<pinref part="C23" gate="G$1" pin="2"/>
-<wire x1="150.114" y1="54.864" x2="150.114" y2="59.436" width="0.1524" layer="91"/>
-<junction x="150.114" y="54.864"/>
-<pinref part="U6" gate="A" pin="S"/>
-<wire x1="140.716" y1="70.612" x2="140.716" y2="59.436" width="0.1524" layer="91"/>
-<wire x1="150.114" y1="59.436" x2="144.018" y2="59.436" width="0.1524" layer="91"/>
-<wire x1="144.018" y1="59.436" x2="140.716" y2="59.436" width="0.1524" layer="91"/>
-<wire x1="144.018" y1="60.452" x2="144.018" y2="59.436" width="0.1524" layer="91"/>
-<pinref part="P+1" gate="VCC" pin="VCC"/>
-</segment>
-<segment>
-<pinref part="BATT_SW" gate="G$1" pin="1"/>
-<wire x1="153.162" y1="98.806" x2="155.448" y2="98.806" width="0.1524" layer="91"/>
-<pinref part="P+3" gate="VCC" pin="VCC"/>
-</segment>
 </net>
 <net name="CBUS1" class="0">
@@
 <wire x1="98.044" y1="120.904" x2="98.044" y2="118.364" width="0.1524" layer="91"/>
 <junction x="95.504" y="120.904"/>
-</segment>
-<segment>
-<pinref part="LED" gate="G$1" pin="K"/>
-<pinref part="SUPPLY2" gate="G$1" pin="3.3V"/>
-<wire x1="120.142" y1="102.87" x2="120.142" y2="101.092" width="0.1524" layer="91"/>
 </segment>
 <segment>
@@
 <pinref part="SUPPLY5" gate="G$1" pin="3.3V"/>
 </segment>
+<segment>
+<pinref part="LED" gate="G$1" pin="A"/>
+<pinref part="SUPPLY2" gate="G$1" pin="3.3V"/>
+<wire x1="120.142" y1="105.156" x2="120.142" y2="101.092" width="0.1524" layer="91"/>
+</segment>
 </net>
 <net name="N$9" class="0">
@@
 <junction x="73.406" y="138.176"/>
 <junction x="72.566" y="138.18"/>
-</segment>
-</net>
-<net name="N$27" class="0">
-<segment>
-<pinref part="LED" gate="G$1" pin="A"/>
-<pinref part="R9" gate="G$1" pin="2"/>
-<wire x1="120.142" y1="118.11" x2="120.142" y2="121.412" width="0.1524" layer="91"/>
 </segment>
 </net>
@@
 </segment>
 </net>
+<net name="V+" class="0">
+<segment>
+<pinref part="D1" gate="G$1" pin="K"/>
+<pinref part="C23" gate="G$1" pin="2"/>
+<wire x1="150.114" y1="54.864" x2="150.114" y2="59.436" width="0.1524" layer="91"/>
+<junction x="150.114" y="54.864"/>
+<pinref part="U6" gate="A" pin="S"/>
+<wire x1="140.716" y1="70.612" x2="140.716" y2="59.436" width="0.1524" layer="91"/>
+<wire x1="150.114" y1="59.436" x2="144.018" y2="59.436" width="0.1524" layer="91"/>
+<wire x1="144.018" y1="59.436" x2="140.716" y2="59.436" width="0.1524" layer="91"/>
+<wire x1="144.018" y1="60.452" x2="144.018" y2="59.436" width="0.1524" layer="91"/>
+<pinref part="P+1" gate="1" pin="V+"/>
+</segment>
+<segment>
+<pinref part="BATT_SW" gate="G$1" pin="1"/>
+<wire x1="153.162" y1="98.806" x2="155.448" y2="98.806" width="0.1524" layer="91"/>
+<pinref part="P+3" gate="1" pin="V+"/>
+</segment>
+</net>
+<net name="N$2" class="0">
+<segment>
+<pinref part="R9" gate="G$1" pin="2"/>
+<pinref part="LED" gate="G$1" pin="K"/>
+<wire x1="120.142" y1="121.412" x2="120.142" y2="120.396" width="0.1524" layer="91"/>
+</segment>
+</net>

Commit message: FIX: fix miss on pcb and update gerber and schematic
Connections:
- removed net N$17: R15.1, U3.TEMP
- net GND: now also R15.1, U3.TEMP
Changed lines of the file:
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@@
 <part name="P+1" library="supply1" library_urn="urn:adsk.eagle:library:371" deviceset="V+" device=""/>
 <part name="P+3" library="supply1" library_urn="urn:adsk.eagle:library:371" deviceset="V+" device=""/>
+<part name="GND6" library="DecawaveLibrary" library_urn="urn:adsk.eagle:library:5224885" deviceset="GND" device=""/>
 </parts>
 <sheets>
@@
 </instance>
 <instance part="IC1" gate="G$1" x="77.724" y="60.706" smashed="yes">
-<attribute name="NAME" x="80.264" y="23.876" size="1.778" layer="95" rot="R90" align="center-left"/>
-<attribute name="VALUE" x="80.264" y="31.496" size="1.778" layer="96" rot="R90" align="center-left"/>
+<attribute name="NAME" x="85.344" y="16.256" size="1.016" layer="95" rot="R180" align="center-left"/>
+<attribute name="VALUE" x="105.41" y="16.002" size="1.016" layer="96" rot="R180" align="center-left"/>
 </instance>
 <instance part="R10" gate="G$1" x="55.88" y="76.454" smashed="yes" rot="R180">
@@
 </instance>
 <instance part="TX" gate="G$1" x="22.86" y="76.454" smashed="yes">
-<attribute name="NAME" x="33.782" y="77.216" size="1.016" layer="95"/>
-<attribute name="VALUE" x="23.368" y="77.47" size="1.016" layer="96"/>
+<attribute name="NAME" x="33.782" y="74.676" size="1.016" layer="95"/>
+<attribute name="VALUE" x="23.368" y="74.676" size="1.016" layer="96"/>
 </instance>
 <instance part="RX" gate="G$1" x="22.86" y="63.754" smashed="yes">
-<attribute name="NAME" x="34.29" y="64.516" size="1.016" layer="95"/>
-<attribute name="VALUE" x="23.368" y="64.77" size="1.016" layer="96"/>
+<attribute name="NAME" x="33.782" y="61.722" size="1.016" layer="95"/>
+<attribute name="VALUE" x="23.368" y="61.976" size="1.016" layer="96"/>
 </instance>
 <instance part="C17" gate="G$1" x="75.184" y="60.706" smashed="yes" rot="R180">
@@
 </instance>
 <instance part="P+1" gate="1" x="144.018" y="62.992" smashed="yes">
-<attribute name="VALUE" x="145.542" y="65.278" size="1.778" layer="96" rot="R180"/>
+<attribute name="VALUE" x="145.034" y="64.516" size="1.016" layer="96" rot="R180"/>
 </instance>
 <instance part="P+3" gate="1" x="150.622" y="98.806" smashed="yes" rot="R90">
-<attribute name="VALUE" x="148.336" y="100.33" size="1.778" layer="96" rot="R270"/>
+<attribute name="VALUE" x="149.606" y="99.822" size="1.778" layer="96" rot="R180"/>
+</instance>
+<instance part="GND6" gate="1" x="186.436" y="122.428" smashed="yes" rot="R270">
+<attribute name="VALUE" x="186.182" y="122.428" size="1.016" layer="96" rot="R270" align="top-center"/>
 </instance>
 </instances>
@@
 <wire x1="240.03" y1="68.58" x2="237.998" y2="68.58" width="0.1524" layer="91"/>
 <pinref part="GND5" gate="1" pin="GND"/>
+</segment>
+<segment>
+<pinref part="U3" gate="G$1" pin="TEMP"/>
+<pinref part="R15" gate="G$1" pin="1"/>
+<wire x1="196.088" y1="112.268" x2="196.088" y2="122.428" width="0.1524" layer="91"/>
+<wire x1="196.088" y1="122.428" x2="188.976" y2="122.428" width="0.1524" layer="91"/>
+<pinref part="GND6" gate="1" pin="GND"/>
+<junction x="188.976" y="122.428"/>
 </segment>
 </net>
@@
 </segment>
 </net>
-<net name="N$17" class="0">
-<segment>
-<pinref part="U3" gate="G$1" pin="TEMP"/>
-<pinref part="R15" gate="G$1" pin="1"/>
-<wire x1="196.088" y1="112.268" x2="196.088" y2="122.428" width="0.1524" layer="91"/>
-<wire x1="196.088" y1="122.428" x2="188.976" y2="122.428" width="0.1524" layer="91"/>
-</segment>
-</net>
